File: pcb/RGB-clock/RGB-clock.sch (KiCad schematic (older format))
At the start: 10 parts, among them P1 FTDI, P2 Display, SW1 Reset, SW2 Flash, U1 ESP-12

Commit message: Updated PCB
Parts:
- C1: symbol C -> Device:C
- P1: symbol CONN_01X06 -> RGB-clock-rescue:CONN_01X06
- P2: symbol CONN_01X03 -> RGB-clock-rescue:CONN_01X03
- R1, R2, R3, R4: symbol R -> Device:R
- SW1, SW2: symbol SW_PUSH -> RGB-clock-rescue:SW_PUSH
- U1: footprint (none) -> ESP8266:ESP-12; symbol ESP-12 -> ESP8266:ESP-12
Changed lines of the file:
@@
-EESchema Schematic File Version 2
-LIBS:power
-LIBS:device
-LIBS:transistors
-LIBS:conn
-LIBS:linear
-LIBS:regul
-LIBS:74xx
-LIBS:cmos4000
-LIBS:adc-dac
-LIBS:memory
-LIBS:xilinx
-LIBS:microcontrollers
-LIBS:dsp
-LIBS:microchip
-LIBS:analog_switches
-LIBS:motorola
-LIBS:texas
-LIBS:intel
-LIBS:audio
-LIBS:interface
-LIBS:digital-audio
-LIBS:philips
-LIBS:display
-LIBS:cypress
-LIBS:siliconi
-LIBS:opto
-LIBS:atmel
-LIBS:contrib
-LIBS:valves
-LIBS:ESP8266
+EESchema Schematic File Version 4
 LIBS:RGB-clock-cache
-EELAYER 25 0
+EELAYER 29 0
 EELAYER END
 $Descr A4 11693 8268
@@
 $EndDescr
 $Comp
-L R R4
+L Device:R R4
 U 1 1 58A755D9
 P 7000 3500
@@
 $EndComp
 $Comp
-L R R3
+L Device:R R3
 U 1 1 58A7564E
 P 6750 4000
@@
 $EndComp
 $Comp
-L R R2
+L Device:R R2
 U 1 1 58A756C8
 P 4500 3350
@@
 $EndComp
 $Comp
-L R R1
+L Device:R R1
 U 1 1 58A75703
 P 4500 3150
@@
 $EndComp
 $Comp
-L +3.3V #PWR6
+L power:+3.3V #PWR06
 U 1 1 58A75922
 P 4300 2650
-F 0 "#PWR6" H 4300 2500 50  0001 C CNN
+F 0 "#PWR06" H 4300 2500 50  0001 C CNN
 F 1 "+3.3V" H 4300 2790 50  0000 C CNN
 F 2 "" H 4300 2650 50  0000 C CNN
@@
 $EndComp
 $Comp
-L GND #PWR9
+L power:GND #PWR09
 U 1 1 58A75940
 P 7000 4750
-F 0 "#PWR9" H 7000 4500 50  0001 C CNN
+F 0 "#PWR09" H 7000 4500 50  0001 C CNN
 F 1 "GND" H 7000 4600 50  0000 C CNN
 F 2 "" H 7000 4750 50  0000 C CNN
@@
 $EndComp
 $Comp
-L CONN_01X06 P1
+L RGB-clock-rescue:CONN_01X06 P1
 U 1 1 58A759A4
 P 7750 3300
@@
 $EndComp
 $Comp
-L +3.3V #PWR8
+L power:+3.3V #PWR08
 U 1 1 58A75D2B
 P 7000 2650
-F 0 "#PWR8" H 7000 2500 50  0001 C CNN
+F 0 "#PWR08" H 7000 2500 50  0001 C CNN
 F 1 "+3.3V" H 7000 2790 50  0000 C CNN
 F 2 "" H 7000 2650 50  0000 C CNN
@@
 $EndComp
 $Comp
-L SW_PUSH SW2
+L RGB-clock-rescue:SW_PUSH SW2
 U 1 1 58A76453
 P 7000 4150
@@
 $EndComp
 $Comp
-L SW_PUSH SW1
+L RGB-clock-rescue:SW_PUSH SW1
 U 1 1 58A765D4
 P 4750 4300
@@
 	7550 3250 6600 3250
 Wire Wire Line
-	4300 2650 4300 4150
+	4300 2650 4300 2750
 Wire Wire Line
 	4300 3350 4350 3350
@@
 Connection ~ 4300 3150
 Wire Wire Line
-	4650 3150 4800 3150
+	4650 3150 4750 3150
 Wire Wire Line
 	4650 3350 4800 3350
@@
 	6750 3750 6750 3850
 Wire Wire Line
-	6600 4650 7550 4650
-Wire Wire Line
-	7000 4450 7000 4750
+	6600 4650 6750 4650
+Wire Wire Line
+	7000 4450 7000 4650
 Wire Wire Line
 	6750 4650 6750 4150
 Connection ~ 6750 4650
 $Comp
-L GND #PWR7
+L power:GND #PWR07
 U 1 1 58A77741
 P 4750 4750
-F 0 "#PWR7" H 4750 4500 50  0001 C CNN
+F 0 "#PWR07" H 4750 4500 50  0001 C CNN
 F 1 "GND" H 4750 4600 50  0000 C CNN
 F 2 "" H 4750 4750 50  0000 C CNN
@@
 NoConn ~ 6600 3350
 $Comp
-L C C1
+L Device:C C1
 U 1 1 58A78796
 P 4300 4300
@@
 	1    0    0    -1
 $EndComp
-Connection ~ 4300 3850
 Wire Wire Line
 	4300 4450 4300 4600
@@
 Connection ~ 7000 4650
 $Comp
-L +3.3V #PWR3
+L power:+3.3V #PWR03
 U 1 1 58A79336
 P 2950 2600
-F 0 "#PWR3" H 2950 2450 50  0001 C CNN
+F 0 "#PWR03" H 2950 2450 50  0001 C CNN
 F 1 "+3.3V" H 2950 2740 50  0000 C CNN
 F 2 "" H 2950 2600 50  0000 C CNN
@@
 $EndComp
 $Comp
-L GND #PWR1
+L power:GND #PWR01
 U 1 1 58A7935C
 P 2150 2600
-F 0 "#PWR1" H 2150 2350 50  0001 C CNN
+F 0 "#PWR01" H 2150 2350 50  0001 C CNN
 F 1 "GND" H 2150 2450 50  0000 C CNN
 F 2 "" H 2150 2600 50  0000 C CNN
@@
 $EndComp
 $Comp
-L PWR_FLAG #FLG1
+L power:PWR_FLAG #FLG01
 U 1 1 58A79477
 P 2150 2450
-F 0 "#FLG1" H 2150 2545 50  0001 C CNN
+F 0 "#FLG01" H 2150 2545 50  0001 C CNN
 F 1 "PWR_FLAG" H 2150 2630 50  0000 C CNN
 F 2 "" H 2150 2450 50  0000 C CNN
@@
 $EndComp
 $Comp
-L PWR_FLAG #FLG3
+L power:PWR_FLAG #FLG03
 U 1 1 58A7952D
 P 2950 2450
-F 0 "#FLG3" H 2950 2545 50  0001 C CNN
+F 0 "#FLG03" H 2950 2545 50  0001 C CNN
 F 1 "PWR_FLAG" H 2950 2630 50  0000 C CNN
 F 2 "" H 2950 2450 50  0000 C CNN
@@
 	7550 4650 7550 3550
 $Comp
-L CONN_01X03 P2
+L RGB-clock-rescue:CONN_01X03 P2
 U 1 1 5B7338E4
 P 3450 3550
@@
 	3650 3550 4800 3550
 $Comp
-L +5V #PWR4
+L power:+5V #PWR04
 U 1 1 5B733A1B
 P 3750 3300
-F 0 "#PWR4" H 3750 3150 50  0001 C CNN
+F 0 "#PWR04" H 3750 3150 50  0001 C CNN
 F 1 "+5V" H 3750 3440 50  0000 C CNN
 F 2 "" H 3750 3300 50  0000 C CNN
@@
 	3750 3450 3650 3450
 $Comp
-L +5V #PWR2
+L power:+5V #PWR02
 U 1 1 5B733A72
 P 2550 2600
-F 0 "#PWR2" H 2550 2450 50  0001 C CNN
+F 0 "#PWR02" H 2550 2450 50  0001 C CNN
 F 1 "+5V" H 2550 2740 50  0000 C CNN
 F 2 "" H 2550 2600 50  0000 C CNN
@@
 $EndComp
 $Comp
-L PWR_FLAG #FLG2
+L power:PWR_FLAG #FLG02
 U 1 1 5B733AA2
 P 2550 2450
-F 0 "#FLG2" H 2550 2545 50  0001 C CNN
+F 0 "#FLG02" H 2550 2545 50  0001 C CNN
 F 1 "PWR_FLAG" H 2550 2630 50  0000 C CNN
 F 2 "" H 2550 2450 50  0000 C CNN
@@
 	2550 2450 2550 2600
 $Comp
-L GND #PWR5
+L power:GND #PWR05
 U 1 1 5B733B06
 P 3750 3800
-F 0 "#PWR5" H 3750 3550 50  0001 C CNN
+F 0 "#PWR05" H 3750 3550 50  0001 C CNN
 F 1 "GND" H 3750 3650 50  0000 C CNN
 F 2 "" H 3750 3800 50  0000 C CNN
@@
 	3750 3650 3750 3800
 $Comp
-L ESP-12 U1
+L ESP8266:ESP-12 U1
 U 1 1 5B7354DD
 P 5700 3450
 F 0 "U1" H 5700 3350 50  0000 C CNN
 F 1 "ESP-12" H 5700 3550 50  0000 C CNN
-F 2 "" H 5700 3450 50  0001 C CNN
+F 2 "ESP8266:ESP-12" H 5700 3450 50  0001 C CNN
 F 3 "" H 5700 3450 50  0001 C CNN
 	1    5700 3450
@@
 Wire Wire Line
 	5700 4350 6600 4350
-Connection ~ 6600 4350
 Wire Wire Line
 	6600 4350 6600 4650
@@
 	5500 2550 5700 2550
 Connection ~ 4300 2750
+Wire Wire Line
+	4300 3150 4300 3350
+Wire Wire Line
+	4750 3150 4800 3150
+Wire Wire Line
+	6750 4650 7000 4650
+Wire Wire Line
+	7000 4650 7000 4750
+Wire Wire Line
+	7000 4650 7550 4650
+Wire Wire Line
+	4300 2750 4300 3150
+Wire Wire Line
+	4300 3350 4300 4150
 $EndSCHEMATC
